Commit message: Added box primitive and changed launch file to Python

File: hand_ws/src/hand_description/urdf/salisbury_hand.urdf.xacro (robot description, xacro)
@@ -26,4 +26,7 @@
   <material name="purple">
     <color rgba="0.5 0 0.5 1.0"/>
+  </material>
+  <material name="green">
+    <color rgba="0.0 1.0 0.0 1.0"/>
   </material>
   <!-- The root link -->
@@ -129,7 +132,66 @@
     </joint>
   </xacro:macro>
+  <!-- Macro definition for a box -->
+  <xacro:macro name="create_fixed_box"
+               params="box_name:='grasp_box'
+                       box_size_x:='0.06'
+                       box_size_y:='0.03'
+                       box_size_z:='0.02'
+                       xyz:='0 0 0'
+                       rpy:='0 0 0'
+                       material_name:='green'">
+    <link name="${box_name}">
+      <visual>
+        <origin xyz="0 0 0" rpy="0 0 0"/>
+        <geometry>
+          <box size="${box_size_x} ${box_size_y} ${box_size_z}"/>
+        </geometry>
+        <material name="${material_name}"/>
+      </visual>
+      <collision>
+        <origin xyz="0 0 0" rpy="0 0 0"/>
+        <geometry>
+          <box size="${box_size_x} ${box_size_y} ${box_size_z}"/>
+        </geometry>
+      </collision>
+      <inertial>
+        <origin xyz="0 0 0" rpy="0 0 0"/>
+        <mass value="0.2"/>
+        <inertia ixx="0.0001" ixy="0.0" ixz="0.0"
+                 iyy="0.0001" iyz="0.0"
+                 izz="0.0001"/>
+      </inertial>
+    </link>
+    <joint name="${box_name}_fixed_joint" type="fixed">
+      <parent link="world"/>
+      <child link="${box_name}"/>
+      <origin xyz="${xyz}" rpy="${rpy}"/>
+    </joint>
+  </xacro:macro>
   <!-- Instantiate fingers -->
-  <xacro:finger finger_id="1" base_xyz="${finger1_base}" invert="false" theta_lower_joint0="${-PI/8}" theta_upper_joint0="${PI/8}"/>
-  <xacro:finger finger_id="2" base_xyz="${finger2_base}" invert="true" theta_lower_joint0="${-PI/8}" theta_upper_joint0="${PI/8}"/>
-  <xacro:finger finger_id="3" base_xyz="${finger3_base}" invert="true" theta_lower_joint0="${-PI/8}" theta_upper_joint0="${PI/8}"/>
+  <xacro:finger finger_id="1"
+                base_xyz="${finger1_base}"
+                invert="false"
+                theta_lower_joint0="${-PI/8}"
+                theta_upper_joint0="${PI/8}"/>
+  <xacro:finger finger_id="2"
+                base_xyz="${finger2_base}"
+                invert="true"
+                theta_lower_joint0="${-PI/8}"
+                theta_upper_joint0="${PI/8}"/>
+  <xacro:finger finger_id="3"
+                base_xyz="${finger3_base}"
+                invert="true"
+                theta_lower_joint0="${-PI/8}"
+                theta_upper_joint0="${PI/8}"/>
+  <!-- Instantiate the box -->
+  <xacro:create_fixed_box
+    box_name="grasp_box"
+    box_size_x="0.06"
+    box_size_y="0.06"
+    box_size_z="0.02"
+    xyz="0.5 0.0 0.05"
+    rpy="0 0 0"
+    material_name="green"
+  />
 </robot>

Commit message: Fix visuals for fingertip

File: hand_ws/src/hand_description/urdf/salisbury_hand.urdf.xacro (robot description, xacro)
@@ -33,7 +33,7 @@
   <link name="world"/>
   <!-- Helper macros for visuals -->
-  <xacro:macro name="vis_sphere" params="radius material">
+  <xacro:macro name="vis_sphere" params="radius material origin_xyz='0 0 0'">
     <visual>
-      <origin xyz="0 0 0" rpy="0 0 0"/>
+      <origin xyz="${origin_xyz}" rpy="0 0 0"/>
       <geometry>
         <sphere radius="${radius}"/>
@@ -124,10 +124,10 @@
     <!-- Fingertip Visual (Sphere) -->
     <link name="finger${finger_id}_tip_visual">
-      <xacro:vis_sphere radius="${r}" material="purple"/>
+      <xacro:vis_sphere radius="${r}" material="purple" origin_xyz="-${r} 0 0"/>
     </link>
     <joint name="finger${finger_id}_tip_fixed" type="fixed">
       <parent link="finger${finger_id}_link2_cylinder"/>
       <child link="finger${finger_id}_tip_visual"/>
-      <origin xyz="${h + r} 0 0"/>
+      <origin xyz="${h + 2*r} 0 0"/>
     </joint>
   </xacro:macro>

Commit message: Added hand control package

File: hand_ws/src/hand_description/urdf/salisbury_hand.urdf.xacro (robot description, xacro)
@@ -163,5 +163,5 @@
       </inertial>
     </link>
-    <joint name="${box_name}_fixed_joint" type="fixed">
+    <joint name="${box_name}_fixed_joint" type="floating">
       <parent link="world"/>
       <child link="${box_name}"/>

Commit message: Returned center of mass joint type to fixed

File: hand_ws/src/hand_description/urdf/salisbury_hand.urdf.xacro (robot description, xacro)
@@ -163,5 +163,5 @@
       </inertial>
     </link>
-    <joint name="${box_name}_fixed_joint" type="floating">
+    <joint name="${box_name}_fixed_joint" type="fixed">
       <parent link="world"/>
       <child link="${box_name}"/>

Commit message: Added contact points frames and parameters for box calculation

File: hand_ws/src/hand_description/urdf/salisbury_hand.urdf.xacro (robot description, xacro)
@@ -17,4 +17,11 @@
   <xacro:property name="r" value="${cylinder_radius}" />
   <xacro:property name="sphere_radius" value="${cylinder_radius*2}" />
+  <xacro:property name="fingertip_x" value="0.267" />
+  <xacro:property name="fingertip_y_range" value="0.10" />
+  <xacro:property name="fingertip_z_range" value="0.034" />
+   <xacro:property name="box_size_y_tolerance" value="0.05" />
+  <xacro:property name="box_size_x" value="0.03" />
+  <xacro:property name="box_size_y" value="${fingertip_y_range + box_size_y_tolerance}" />
+  <xacro:property name="box_size_z" value="${fingertip_z_range - 2*r}" />
   <!-- Global Materials -->
   <material name="sky_blue">
@@ -53,5 +60,4 @@
   <!-- Macro to create a finger chain -->
   <xacro:macro name="finger" params="finger_id base_xyz invert theta_lower_joint0 theta_upper_joint0">
-    <!-- Base Joint Visual (Sphere) -->
     <link name="finger${finger_id}_base_joint">
       <xacro:vis_sphere radius="${sphere_radius}" material="sky_blue"/>
@@ -62,5 +68,4 @@
       <origin xyz="${base_xyz}" rpy="${(PI if invert else 0)} ${(-PI/4 if invert else PI/4)} 0"/>
     </joint>
-    <!-- Joint0 Visual (Sphere) -->
     <link name="finger${finger_id}_joint0_visual">
       <xacro:vis_sphere radius="${sphere_radius}" material="sky_blue"/>
@@ -72,5 +77,4 @@
       <limit lower="${theta_lower_joint0}" upper="${theta_upper_joint0}" effort="10" velocity="1"/>
     </joint>
-    <!-- Link0 (Cylinder) -->
     <link name="finger${finger_id}_link0_cylinder">
       <xacro:vis_cylinder length="${a1}" radius="${cylinder_radius}" material="dark_blue"
@@ -82,5 +86,4 @@
       <origin xyz="${a1} 0 0" rpy="${-PI/2} 0 0"/>
     </joint>
-    <!-- Joint1 Visual (Sphere) -->
     <link name="finger${finger_id}_joint1_visual">
       <xacro:vis_sphere radius="${sphere_radius}" material="sky_blue"/>
@@ -92,5 +95,4 @@
       <limit lower="${-PI/4}" upper="${-PI/2}" effort="10" velocity="1"/>
     </joint>
-    <!-- Link1 (Cylinder) -->
     <link name="finger${finger_id}_link1_cylinder">
       <xacro:vis_cylinder length="${a2}" radius="${cylinder_radius}" material="dark_blue"
@@ -102,5 +104,4 @@
       <origin xyz="${a2} 0 0"/>
     </joint>
-    <!-- Joint2 Visual (Sphere) -->
     <link name="finger${finger_id}_joint2_visual">
       <xacro:vis_sphere radius="${sphere_radius}" material="sky_blue"/>
@@ -112,5 +113,4 @@
       <limit lower="${-PI/16}" upper="${-PI/4}" effort="10" velocity="1"/>
     </joint>
-    <!-- Link2 (Cylinder) -->
     <link name="finger${finger_id}_link2_cylinder">
       <xacro:vis_cylinder length="${a3 + h}" radius="${cylinder_radius}" material="dark_blue"
@@ -122,5 +122,4 @@
       <origin xyz="${a3} 0 0"/>
     </joint>
-    <!-- Fingertip Visual (Sphere) -->
     <link name="finger${finger_id}_tip_visual">
       <xacro:vis_sphere radius="${r}" material="purple" origin_xyz="-${r} 0 0"/>
@@ -188,10 +187,31 @@
   <xacro:create_fixed_box
     box_name="grasp_box"
-    box_size_x="0.01"
-    box_size_y="0.10"
-    box_size_z="${0.034 - 2*r}"
-    xyz="0.267 0 0"
+    box_size_x="${box_size_x}"
+    box_size_y="${box_size_y}"
+    box_size_z="${box_size_z}"
+    xyz="${fingertip_x} 0 0"
     rpy="0 0 0"
     material_name="green"
   />
+  <!-- Finger 1 contact reference frame on the box -->
+  <link name="finger1_box_contact_frame"/>
+  <joint name="finger1_box_contact_frame_joint" type="fixed">
+    <parent link="grasp_box"/>
+    <child link="finger1_box_contact_frame"/>
+    <origin xyz="0.006 0.000 -0.009" rpy="-1.571 -0.884 0.000"/>
+  </joint>
+  <!-- Finger 2 contact reference frame on the box -->
+  <link name="finger2_box_contact_frame"/>
+  <joint name="finger2_box_contact_frame_joint" type="fixed">
+    <parent link="grasp_box"/>
+    <child link="finger2_box_contact_frame"/>
+    <origin xyz="0.007 -0.050 0.009" rpy="1.571 0.880 0.000"/>
+  </joint>
+  <!-- Finger 3 contact reference frame on the box -->
+  <link name="finger3_box_contact_frame"/>
+  <joint name="finger3_box_contact_frame_joint" type="fixed">
+    <parent link="grasp_box"/>
+    <child link="finger3_box_contact_frame"/>
+    <origin xyz="0.006 0.050 0.009" rpy="1.571 0.885 0.000"/>
+  </joint>
 </robot>

Commit message: Add URDF feature to allow the box move with 6DOF

File: hand_ws/src/hand_description/urdf/salisbury_hand.urdf.xacro (robot description, xacro)
@@ -132,5 +132,5 @@
   </xacro:macro>
   <!-- Macro definition for a box -->
-  <xacro:macro name="create_fixed_box"
+  <!-- <xacro:macro name="create_fixed_box"
                params="box_name
                        box_size_x
@@ -167,4 +167,33 @@
       <origin xyz="${xyz}" rpy="${rpy}"/>
     </joint>
+  </xacro:macro> -->
+  <!-- Macro para crear la caja sin joint fijo (solo el link) -->
+  <xacro:macro name="create_floating_box"
+               params="box_name
+                       box_size_x
+                       box_size_y
+                       box_size_z">
+    <link name="${box_name}">
+      <visual>
+        <origin xyz="0 0 0" rpy="0 0 0"/>
+        <geometry>
+          <box size="${box_size_x} ${box_size_y} ${box_size_z}"/>
+        </geometry>
+        <material name="green"/>
+      </visual>
+      <collision>
+        <origin xyz="0 0 0" rpy="0 0 0"/>
+        <geometry>
+          <box size="${box_size_x} ${box_size_y} ${box_size_z}"/>
+        </geometry>
+      </collision>
+      <inertial>
+        <origin xyz="0 0 0" rpy="0 0 0"/>
+        <mass value="0.2"/>
+        <inertia ixx="0.0001" ixy="0.0" ixz="0.0"
+                 iyy="0.0001" iyz="0.0"
+                 izz="0.0001"/>
+      </inertial>
+    </link>
   </xacro:macro>
   <!-- Instantiate the 3 fingers -->
@@ -185,5 +214,5 @@
                 theta_upper_joint0="${PI/8}"/>
   <!-- Box that encloses the three fingertip coords when joints centered -->
-  <xacro:create_fixed_box
+  <!-- <xacro:create_fixed_box
     box_name="grasp_box"
     box_size_x="${box_size_x}"
@@ -193,5 +222,65 @@
     rpy="0 0 0"
     material_name="green"
-  />
+  /> -->
+  <!-- Definición de la caja con 6 DOF mediante joints dummy -->
+  <!-- 1) Se fija la posición base de la caja con el offset deseado -->
+  <joint name="grasp_box_base_fixed" type="fixed">
+    <parent link="world"/>
+    <child link="grasp_box_base"/>
+    <origin xyz="${fingertip_x} 0 0" rpy="0 0 0"/>
+  </joint>
+  <link name="grasp_box_base"/>
+  <!-- 2) Se crea el link de la caja (visual, colisión, inercia) -->
+  <xacro:create_floating_box box_name="grasp_box" box_size_x="${box_size_x}" box_size_y="${box_size_y}" box_size_z="${box_size_z}"/>
+  <!-- 3) Cadena dummy de joints para otorgar 6 DOF a partir del frame base -->
+  <!-- Traslaciones -->
+  <joint name="grasp_box_trans_x" type="prismatic">
+    <parent link="grasp_box_base"/>
+    <child link="grasp_box_trans_x_link"/>
+    <origin xyz="0 0 0" rpy="0 0 0"/>
+    <axis xyz="1 0 0"/>
+    <limit lower="-1" upper="1" effort="10" velocity="1"/>
+  </joint>
+  <link name="grasp_box_trans_x_link"/>
+  <joint name="grasp_box_trans_y" type="prismatic">
+    <parent link="grasp_box_trans_x_link"/>
+    <child link="grasp_box_trans_y_link"/>
+    <origin xyz="0 0 0" rpy="0 0 0"/>
+    <axis xyz="0 1 0"/>
+    <limit lower="-1" upper="1" effort="10" velocity="1"/>
+  </joint>
+  <link name="grasp_box_trans_y_link"/>
+  <joint name="grasp_box_trans_z" type="prismatic">
+    <parent link="grasp_box_trans_y_link"/>
+    <child link="grasp_box_trans_z_link"/>
+    <origin xyz="0 0 0" rpy="0 0 0"/>
+    <axis xyz="0 0 1"/>
+    <limit lower="-1" upper="1" effort="10" velocity="1"/>
+  </joint>
+  <link name="grasp_box_trans_z_link"/>
+  <!-- Rotaciones -->
+  <joint name="grasp_box_rot_x" type="revolute">
+    <parent link="grasp_box_trans_z_link"/>
+    <child link="grasp_box_rot_x_link"/>
+    <origin xyz="0 0 0" rpy="0 0 0"/>
+    <axis xyz="1 0 0"/>
+    <limit lower="-3.14" upper="3.14" effort="10" velocity="1"/>
+  </joint>
+  <link name="grasp_box_rot_x_link"/>
+  <joint name="grasp_box_rot_y" type="revolute">
+    <parent link="grasp_box_rot_x_link"/>
+    <child link="grasp_box_rot_y_link"/>
+    <origin xyz="0 0 0" rpy="0 0 0"/>
+    <axis xyz="0 1 0"/>
+    <limit lower="-3.14" upper="3.14" effort="10" velocity="1"/>
+  </joint>
+  <link name="grasp_box_rot_y_link"/>
+  <joint name="grasp_box_rot_z" type="revolute">
+    <parent link="grasp_box_rot_y_link"/>
+    <child link="grasp_box"/>
+    <origin xyz="0 0 0" rpy="0 0 0"/>
+    <axis xyz="0 0 1"/>
+    <limit lower="-3.14" upper="3.14" effort="10" velocity="1"/>
+  </joint>
   <!-- Finger 1 contact reference frame on the box -->
   <link name="finger1_box_contact_frame"/>

Commit message: Update rotation of contact point in box object

File: hand_ws/src/hand_description/urdf/salisbury_hand.urdf.xacro (robot description, xacro)
@@ -288,5 +288,6 @@
     <parent link="grasp_box"/>
     <child link="finger1_box_contact_frame"/>
-    <origin xyz="0.006 0.000 -0.009" rpy="-1.571 -0.884 0.000"/>
+    <origin xyz="0.006 0.000 -0.009" rpy="0.0 0.0 0.0"/>
+    <!-- <origin xyz="0.006 0.000 -0.009" rpy="-1.571 -0.884 0.000"/> -->
   </joint>
   <!-- Finger 2 contact reference frame on the box -->
@@ -295,5 +296,6 @@
     <parent link="grasp_box"/>
     <child link="finger2_box_contact_frame"/>
-    <origin xyz="0.007 -0.050 0.009" rpy="1.571 0.880 0.000"/>
+    <origin xyz="0.007 -0.050 0.009" rpy="0.0 0.0 0.0"/>
+    <!-- <origin xyz="0.007 -0.050 0.009" rpy="1.571 0.880 0.000"/> -->
   </joint>
   <!-- Finger 3 contact reference frame on the box -->
@@ -302,5 +304,6 @@
     <parent link="grasp_box"/>
     <child link="finger3_box_contact_frame"/>
-    <origin xyz="0.006 0.050 0.009" rpy="1.571 0.885 0.000"/>
+    <origin xyz="0.006 0.050 0.009" rpy="0.0 0.0 0.0"/>
+    <!-- <origin xyz="0.006 0.050 0.009" rpy="1.571 0.885 0.000"/> -->
   </joint>
 </robot>

Commit message: Corrected format of urdf file

File: hand_ws/src/hand_description/urdf/salisbury_hand.urdf.xacro (robot description, xacro)
@@ -20,5 +20,5 @@
   <xacro:property name="fingertip_y_range" value="0.10" />
   <xacro:property name="fingertip_z_range" value="0.034" />
-   <xacro:property name="box_size_y_tolerance" value="0.05" />
+  <xacro:property name="box_size_y_tolerance" value="0.05" />
   <xacro:property name="box_size_x" value="0.03" />
   <xacro:property name="box_size_y" value="${fingertip_y_range + box_size_y_tolerance}" />
@@ -131,42 +131,5 @@
     </joint>
   </xacro:macro>
-  <!-- Macro definition for a box -->
-  <!-- <xacro:macro name="create_fixed_box"
-               params="box_name
-                       box_size_x
-                       box_size_y
-                       box_size_z
-                       xyz
-                       rpy
-                       material_name">
-    <link name="${box_name}">
-      <visual>
-        <origin xyz="0 0 0" rpy="0 0 0"/>
-        <geometry>
-          <box size="${box_size_x} ${box_size_y} ${box_size_z}"/>
-        </geometry>
-        <material name="${material_name}"/>
-      </visual>
-      <collision>
-        <origin xyz="0 0 0" rpy="0 0 0"/>
-        <geometry>
-          <box size="${box_size_x} ${box_size_y} ${box_size_z}"/>
-        </geometry>
-      </collision>
-      <inertial>
-        <origin xyz="0 0 0" rpy="0 0 0"/>
-        <mass value="0.2"/>
-        <inertia ixx="0.0001" ixy="0.0" ixz="0.0"
-                 iyy="0.0001" iyz="0.0"
-                 izz="0.0001"/>
-      </inertial>
-    </link>
-    <joint name="${box_name}_fixed_joint" type="fixed">
-      <parent link="world"/>
-      <child link="${box_name}"/>
-      <origin xyz="${xyz}" rpy="${rpy}"/>
-    </joint>
-  </xacro:macro> -->
-  <!-- Macro para crear la caja sin joint fijo (solo el link) -->
+  <!-- Macro to create the box without a fixed joint (link only) -->
   <xacro:macro name="create_floating_box"
                params="box_name
@@ -213,16 +176,16 @@
                 theta_lower_joint0="${-PI/8}"
                 theta_upper_joint0="${PI/8}"/>
-  <!-- Box that encloses the three fingertip coords when joints centered -->
+  <!-- Box that encloses the three fingertip coordinates when joints are centered -->
   <!-- <xacro:create_fixed_box
-    box_name="grasp_box"
-    box_size_x="${box_size_x}"
-    box_size_y="${box_size_y}"
-    box_size_z="${box_size_z}"
-    xyz="${fingertip_x} 0 0"
-    rpy="0 0 0"
-    material_name="green"
+       box_name="grasp_box"
+       box_size_x="${box_size_x}"
+       box_size_y="${box_size_y}"
+       box_size_z="${box_size_z}"
+       xyz="${fingertip_x} 0 0"
+       rpy="0 0 0"
+       material_name="green"
   /> -->
-  <!-- Definición de la caja con 6 DOF mediante joints dummy -->
-  <!-- 1) Se fija la posición base de la caja con el offset deseado -->
+  <!-- Definition of the box with 6 DOF using dummy joints -->
+  <!-- 1) Fix the box base position with the desired offset -->
   <joint name="grasp_box_base_fixed" type="fixed">
     <parent link="world"/>
@@ -231,8 +194,8 @@
   </joint>
   <link name="grasp_box_base"/>
-  <!-- 2) Se crea el link de la caja (visual, colisión, inercia) -->
+  <!-- 2) Create the box link (visual, collision, inertia) -->
   <xacro:create_floating_box box_name="grasp_box" box_size_x="${box_size_x}" box_size_y="${box_size_y}" box_size_z="${box_size_z}"/>
-  <!-- 3) Cadena dummy de joints para otorgar 6 DOF a partir del frame base -->
-  <!-- Traslaciones -->
+  <!-- 3) Dummy joint chain to provide 6 DOF from the base frame -->
+  <!-- Translations -->
   <joint name="grasp_box_trans_x" type="prismatic">
     <parent link="grasp_box_base"/>
@@ -259,5 +222,5 @@
   </joint>
   <link name="grasp_box_trans_z_link"/>
-  <!-- Rotaciones -->
+  <!-- Rotations -->
   <joint name="grasp_box_rot_x" type="revolute">
     <parent link="grasp_box_trans_z_link"/>
@@ -289,5 +252,4 @@
     <child link="finger1_box_contact_frame"/>
     <origin xyz="0.006 0.000 -0.009" rpy="0.0 0.0 0.0"/>
-    <!-- <origin xyz="0.006 0.000 -0.009" rpy="-1.571 -0.884 0.000"/> -->
   </joint>
   <!-- Finger 2 contact reference frame on the box -->
@@ -297,5 +259,4 @@
     <child link="finger2_box_contact_frame"/>
     <origin xyz="0.007 -0.050 0.009" rpy="0.0 0.0 0.0"/>
-    <!-- <origin xyz="0.007 -0.050 0.009" rpy="1.571 0.880 0.000"/> -->
   </joint>
   <!-- Finger 3 contact reference frame on the box -->
@@ -305,5 +266,4 @@
     <child link="finger3_box_contact_frame"/>
     <origin xyz="0.006 0.050 0.009" rpy="0.0 0.0 0.0"/>
-    <!-- <origin xyz="0.006 0.050 0.009" rpy="1.571 0.885 0.000"/> -->
   </joint>
 </robot>
